File: hardware/sensor_board/sensor_board.kicad_sch (KiCad schematic)
At the start: 25 parts, among them J1 CORTEX-SWD-6, J2 Molex PicoBlade 1x4, Q1 SI2337DS-T1-BE3, Q2 SI2337DS-T1-BE3, U1 ATSAMC21E17A, U2 TCAN332G, Y1 Crystal

Commit message: updated pcb
Parts:
- added C26: 100nF / 6.3V, Capacitor_SMD:C_0402_1005Metric, symbol Device:C
- added C27: 10uF / 6.3V, Capacitor_SMD:C_0603_1608Metric, symbol Device:C
- C1, C8: value 10u / 6.3V -> 10uF / 6.3V
- C2, C3, C7: value 100n / 50V -> 100nF / 6.3V; footprint Capacitor_SMD:C_0603_1608Metric -> Capacitor_SMD:C_0402_1005Metric
- C25: renamed from C?; footprint Capacitor_SMD:C_0603_1608Metric -> Capacitor_SMD:C_0402_1005Metric
- C4, C5: value 18p -> 15pF / 6.3V; footprint Capacitor_SMD:C_0603_1608Metric -> Capacitor_SMD:C_0402_1005Metric
- C6: value 1u / 6.3V -> 1uF / 6.3V
- R1, R2, R3, R4, R5: footprint Resistor_SMD:R_0603_1608Metric -> Resistor_SMD:R_0402_1005Metric
- R7, R8: renamed from R?; footprint Resistor_SMD:R_0603_1608Metric -> Resistor_SMD:R_0402_1005Metric
Connections:
- net GND: now also J1.2 (GND), C26.2, C27.2; no longer J1.5 (GND)
- net SWCLK: now also J1.3 (SWCLK); no longer J1.4 (SWCLK)
- net SWDIO: now also J1.5 (SWDIO); no longer J1.2 (SWDIO)
- net VDD: now also J1.6 (VCC), C26.1, C27.1; no longer J1.1 (VCC)
- net VDDSW_SIG: now also U1.3 (PA02); no longer U1.5 (PA04)
- net ~{RESET}: now also J1.4 (~{RESET}); no longer J1.3 (nRESET)
- net SERCOM0.2: now reaches U1.7 (PA06)
- net SERCOM0.3: now reaches U1.8 (PA07)
- net CO2CAL renamed SERCOM0.1
- net UART.RX renamed GPIO.1
- net UART.TX renamed GPIO.0
- new net SERCOM0.0: U1.5 (PA04)
- no-connect marks 14 -> 11
Other:
- sheet Sensors ports: added GPIO{0,1}, SERCOM0{0,1,2,3}; removed CalibrateCO2, UART_{RX}, UART_{TX}
- note added: "Calculate Cs correctly! Parasitic: Xin 5.9 pF Xout 3.1 pF Crystal needs 18pF -> 18 - 6 = 12pF -> 18 - 3 = 15pF 12 + (15 - 12) / 2 = 13.5 -> 15pF"
- note removed: "Calculate Cs correctly! Parasitic: Xin 5.9 pF Xout 3.1 pF"
- note removed: "Pins wrong! Right pins: 1 SWO 2 GND 3 SWCLK 5 SWDIO 4 ~{RESET} 6 3.3V"

Commit message: updated pcb
Parts:
- removed C3: 100nF / 6.3V, Capacitor_SMD:C_0402_1005Metric, symbol Device:C
- removed C4, C5: 15pF / 6.3V, Capacitor_SMD:C_0402_1005Metric, symbol Device:C
- removed J2: Molex PicoBlade 1x4, Connector_Molex:Molex_PicoBlade_53261-0471_1x04-1MP_P1.25mm_Horizontal, symbol Connector:Conn_01x04_Male
- removed Y1: Crystal, ownLib:Abracon_ABC2, symbol Device:Crystal
- added C6: 100nF / 6.3V, Capacitor_SMD:C_0402_1005Metric, symbol Device:C
- added J2: Conn_01x04_MountingPin, Connector_Molex:Molex_PicoBlade_53261-0471_1x04-1MP_P1.25mm_Horizontal, symbol Connector_Generic_MountingPin:Conn_01x04_MountingPin
- added TP1: TestPoint, TestPoint:TestPoint_Keystone_5015_Micro-Minature, symbol Connector:TestPoint
- added Y1: Resonator, Crystal:Resonator_SMD_Murata_CSTxExxV-3Pin_3.0x1.1mm, symbol Device:Resonator
- renumbered C25 to C1, C1 to C2, C2 to C3, C7 to C4, C6 to C5, C8 to C7, C26 to C8, C27 to C9, Q2 to Q1, Q1 to Q2, R7 to R2, R8 to R3, R3 to R4, R2 to R5, R5 to R6, R4 to R7, R6 to R8
Connections:
- net +36V: now also J2.2 (Pin_2)
- net 5VSW_SIG: now also U1.3 (PA02); no longer U1.4 (PA03)
- net CAN+: now also J2.4 (Pin_4)
- net CAN-: now also J2.3 (Pin_3)
- net GND: now also C6.2, J2.1 (Pin_1), J2.MP (MountPin), TP1.1, Y1.2
- net VDD: now also C6.1
- net VDDSW_SIG: now also U1.4 (PA03); no longer U1.3 (PA02)
- net X_{IN}: now also Y1.1
- net X_{OUT}: now also Y1.3
Other:
- note removed: "Calculate Cs correctly! Parasitic: Xin 5.9 pF Xout 3.1 pF Crystal needs 18pF -> 18 - 6 = 12pF -> 18 - 3 = 15pF 12 + (15 - 12) / 2 = 13.5 -> 15pF"
