File: hardware/sensor_board/sensor_board.kicad_pcb (KiCad board)
At the start: 4 copper layers, 66.6 x 34 mm, 50 parts, among them J1 CORTEX-SWD-6, J2 Molex PicoBlade 1x4, J3 Molex PicoBlade 1x7, Q1 SI2337DS-T1-BE3, Q2 SI2337DS-T1-BE3, U1 ATSAMC21E17A, U2 TCAN332G, U3 LMZM23600V3, U4 SHT30-DIS, U5 BMP384, U6 SCD4x, U7 SGP30, U8 BH1751FVI, U9 LMZM23600V5, Y1 Crystal

Commit message: updated pcb
Parts:
- removed C10: 4u7 / 50V, Capacitor_SMD:C_0805_2012Metric
- removed C12, C13: 10u / 10V, Capacitor_SMD:C_0603_1608Metric
- removed H1, H2, H3, H4: MountingHole, MountingHole:MountingHole_3.2mm_M3
- added C25: 10nF / 6.3V, Capacitor_SMD:C_0402_1005Metric, F.Cu at (141.5, 109.3)
- added C26: 100nF / 6.3V, Capacitor_SMD:C_0402_1005Metric, F.Cu at (131.0, 97.5)
- added C27: 10uF / 6.3V, Capacitor_SMD:C_0603_1608Metric, F.Cu at (130.1, 94.6)
- added C28: 100nF / 6.3V, Capacitor_SMD:C_0402_1005Metric, F.Cu at (126.7, 108.7)
- added C29: 10uF / 6.3V, Capacitor_SMD:C_0603_1608Metric, F.Cu at (128.8, 108.5)
- added R7: 10k, Resistor_SMD:R_0402_1005Metric, F.Cu at (149.6, 109.4)
- added R8: 100k, Resistor_SMD:R_0402_1005Metric, F.Cu at (149.6, 111.4)
- C1, C8: value 10u / 10V -> 10uF / 6.3V
- C11: value 10u / 10V -> 1uF / 6.3V
- C14, C15, C16, C17, C18, C19: value 100nF / 10V -> 100nF / 6.3V; footprint Capacitor_SMD:C_0603_1608Metric -> Capacitor_SMD:C_0402_1005Metric
- C2, C3, C7: value 100n / 10V -> 100nF / 6.3V; footprint Capacitor_SMD:C_0603_1608Metric -> Capacitor_SMD:C_0402_1005Metric
- C22, C23, C24: value 10u / 10V -> 10uF / 6.3V; footprint Capacitor_SMD:C_0603_1608Metric -> Capacitor_SMD:C_0402_1005Metric
- C4, C5: value 18p -> 15pF / 6.3V; footprint Capacitor_SMD:C_0603_1608Metric -> Capacitor_SMD:C_0402_1005Metric
- C6: value 1u / 10V -> 1uF / 6.3V
- C9: value 4u7 / 50V -> 1uF / 6.3V; footprint Capacitor_SMD:C_0805_2012Metric -> Capacitor_SMD:C_0603_1608Metric
- J3: footprint Connector_Molex:Molex_PicoBlade_53261-0771_1x07-1MP_P1.25mm_Horizontal -> Connector_Molex:Molex_PicoBlade_53261-1071_1x10-1MP_P1.25mm_Horizontal
- R1: value 2k2 -> 10k; footprint Resistor_SMD:R_0603_1608Metric -> Resistor_SMD:R_0402_1005Metric
- R2, R3, R4, R5: footprint Resistor_SMD:R_0603_1608Metric -> Resistor_SMD:R_0402_1005Metric
- U3: value LMZM23600V3 -> NCP718xSN330; footprint Package_LGA:Texas_SIL0010A_MicroSiP-10-1EP_3.8x3mm_P0.6mm_EP0.7x2.9mm_ThermalVias -> Package_TO_SOT_SMD:SOT-23-5
- moved U4 32.1 mm to (130.8, 104.3)
- moved C16 31.4 mm to (131.4, 106.3)
- moved C17 27.3 mm to (135.2, 109.1), turned to 180 degrees
- moved U7 26.2 mm to (138.6, 108.5), turned to 180 degrees
- moved C18 22.5 mm to (135.4, 106.2), turned to 180 degrees
- moved C19 21.9 mm to (136.3, 103.0)
- moved U8 20.0 mm to (137.1, 105.1), turned to 90 degrees
- moved C15 14.5 mm to (137.7, 106.2), turned to 180 degrees
- moved U5 13.3 mm to (139.9, 105.1)
- moved J3 12.2 mm to (158.4, 97.0)
- moved C14 12.2 mm to (140.9, 103.3)
- moved J1 11.1 mm to (146.5, 107.4), turned to -90 degrees
- moved Q1 9.64 mm to (152.2, 90.5), turned to -90 degrees
- moved U6 9.59 mm to (120.9, 106.9)
- moved C9 8.94 mm to (128.0, 89.8), turned to 180 degrees
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Connections:
- J1 pad 1: VDD -> unconnected-(J1-Pad1)
- J1 pad 2: /SWDIO -> GND
- J1 pad 3: ~{RESET} -> /SWCLK
- J1 pad 4: /SWCLK -> ~{RESET}
- J1 pad 5: GND -> /SWDIO
- J1 pad 6: unconnected-(J1-Pad6) -> VDD
- J2 pad 1: +36V -> GND
- J2 pad 2: GND -> +36V
- J3 pad 1: /CO2CAL -> GND
- J3 pad 2: unconnected-(J3-Pad2) -> /SERCOM0.0
- J3 pad 3: GND -> /SERCOM0.1
- J3 pad 4: /5VSW -> /SERCOM0.2
- J3 pad 5: /UART.RX -> /SERCOM0.3
- J3 pad 6: /UART.TX -> GND
- J3 pad 7: unconnected-(J3-Pad7) -> /VDDSW
- U1 pad 1: /UART.TX -> /GPIO.0
- U1 pad 2: /UART.RX -> /GPIO.1
- U1 pad 3: unconnected-(U1-Pad3) -> /VDDSW_SIG
- U1 pad 5: /VDDSW_SIG -> /SERCOM0.0
- U1 pad 6: /CO2CAL -> /SERCOM0.1
- U1 pad 7: unconnected-(U1-Pad7) -> /SERCOM0.2
- U1 pad 8: unconnected-(U1-Pad8) -> /SERCOM0.3
- U3 pad 1: GND -> +5V
- U3 pad 4: +5V -> unconnected-(U3-Pad4)
- U3 pad 5: unconnected-(U3-Pad5) -> VDD
- U4 pad 2: /VDDSW -> GND
- U7 pad 7: GND -> (no net)
- U8 pad 2: /VDDSW -> GND
Routing:
- net /VDDSW: track 0.00 -> 85.7 mm, vias 0 -> 2
- net VDD: track 0.00 -> 85.5 mm, vias 0 -> 3
- net /I2C.SDA: track 0.00 -> 54.5 mm, vias 0 -> 6
- net /I2C.SCL: track 0.00 -> 49.9 mm, vias 0 -> 6
- net +5V: track 0.00 -> 46.1 mm
- net ~{RESET}: track 0.00 -> 26.3 mm
- net /CAN_{RX}: track 0.00 -> 21.5 mm
- net /CAN_{TX}: track 0.00 -> 21.4 mm
- net /SWDIO: track 0.00 -> 17.3 mm
- net /VDDSW_SIG: track 0.00 -> 15.7 mm, vias 0 -> 2
- net /5VSW_SIG: track 0.00 -> 15.5 mm, vias 0 -> 2
- net /SWCLK: track 0.00 -> 15.4 mm
- net /CAN+: track 0.00 -> 15.0 mm
- net /GPIO.1: track 0.00 -> 13.4 mm, vias 0 -> 2
- net /GPIO.0: track 0.00 -> 12.9 mm, vias 0 -> 2
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- added copper zone on F.Cu, net +36V
- added copper zone on F.Cu, net +5V
- added copper zone on B.Cu, net GND
- added copper zone on F.Cu, net GND
- added copper zone on In1.Cu, net GND
- added copper zone on In2.Cu, net GND
Other:
- board size 66.6 x 34 mm -> 54 x 34 mm

Commit message: updated pcb
Parts:
- removed the C3 at (145.9, 100.1)
- removed the C4 at (142.2, 85.4)
- removed the C5 at (135.6, 85.4)
- added C22: 100nF / 6.3V, Capacitor_SMD:C_0402_1005Metric, F.Cu at (38.7, 7.69)
- added C23: 100nF / 6.3V, Capacitor_SMD:C_0402_1005Metric, F.Cu at (28.2, 16.1)
- added C6: 100nF / 6.3V, Capacitor_SMD:C_0402_1005Metric, F.Cu at (26.8, 23.6)
- added REF**: MountingHole_3.2mm_M3, MountingHole:MountingHole_3.2mm_M3, F.Cu at (3.50, 30.5)
- added REF**: MountingHole_3.2mm_M3, MountingHole:MountingHole_3.2mm_M3, F.Cu at (46.5, 30.5)
- added REF**: MountingHole_3.2mm_M3, MountingHole:MountingHole_3.2mm_M3, F.Cu at (46.5, 3.50)
- added REF**: MountingHole_3.2mm_M3, MountingHole:MountingHole_3.2mm_M3, F.Cu at (3.50, 3.50)
- added TP1: TestPoint, TestPoint:TestPoint_Keystone_5015_Micro-Minature, F.Cu at (24.4, 14.0)
- C12: renamed from C9; value 1uF / 6.3V -> 1uF / 10V
- C14: renamed from C22; value 10uF / 6.3V -> 10uF / 10V
- C15: renamed from C23; value 10uF / 6.3V -> 10uF / 10V
- C16: renamed from C24; value 10uF / 6.3V -> 10uF / 10V
- J2: value Molex PicoBlade 1x4 -> Conn_01x04_MountingPin
- J3: value Molex PicoBlade 1x7 -> Conn_01x10_MountingPin
- Y1: value Crystal -> Resonator; footprint ownLib:Abracon_ABC2 -> Crystal:Resonator_SMD_Murata_CSTxExxV-3Pin_3.0x1.1mm
- moved R2 155.7 mm to (17.4, 27.3)
- moved R3 155.7 mm to (17.4, 29.3)
- moved C1 155.6 mm to (9.21, 27.3)
- moved R1 155.6 mm to (9.60, 25.8)
- moved J1 155.6 mm to (14.3, 25.3)
- moved U8 145.0 mm to (28.6, 14.0), turned to 90 degrees
- moved C2 145.0 mm to (26.9, 20.1), turned to 180 degrees
- moved C12 144.7 mm to (10.4, 5.50), turned to -90 degrees
- moved C21 144.3 mm to (25.7, 7.60), turned to -90 degrees
- moved C24 144.0 mm to (29.0, 11.9), turned to 0 degrees
- moved U3 142.2 mm to (13.3, 6.00)
- moved C20 142.0 mm to (27.0, 7.60)
- moved C7 139.6 mm to (26.8, 22.3), turned to 180 degrees
- moved C5 139.1 mm to (23.9, 32.2), turned to 180 degrees
- moved C3 138.8 mm to (25.9, 31.4), turned to -90 degrees
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- renumbered C25 to C1, C20 to C10, C21 to C11, C11 to C13, C14 to C17, C15 to C18, C16 to C19, C1 to C2, C28 to C20, C29 to C21, C17 to C24, C18 to C25, C19 to C26, C2 to C3, C7 to C4, C6 to C5, C8 to C7, C26 to C8, C27 to C9, Q2 to Q1, Q1 to Q2, R7 to R2, R8 to R3, R3 to R4, R2 to R5, R5 to R6, R4 to R7, R6 to R8, U9 to U4, U4 to U5, U5 to U6, U6 to U7, U7 to U8, U8 to U9
Connections:
- J2 pad 3: /CAN+ -> /CAN-
- J2 pad 4: /CAN- -> /CAN+
- J2 pad MP: (no net) -> GND
- J3 pad 10: /GPIO.1 -> GND
- J3 pad 2: /SERCOM0.0 -> /GPIO.0
- J3 pad 3: /SERCOM0.1 -> /GPIO.1
- J3 pad 4: /SERCOM0.2 -> /VDDSW
- J3 pad 5: /SERCOM0.3 -> /5VSW
- J3 pad 6: GND -> /SERCOM0.0
- J3 pad 7: /VDDSW -> /SERCOM0.1
- J3 pad 8: /5VSW -> /SERCOM0.2
- J3 pad 9: /GPIO.0 -> /SERCOM0.3
- J3 pad MP: (no net) -> GND
- U1 pad 3: /VDDSW_SIG -> /5VSW_SIG
- U1 pad 4: /5VSW_SIG -> /VDDSW_SIG
- U5 pad 6: ~{RESET} -> /VDDSW
- U8 pad 7: (no net) -> GND
- Y1 pad 1: /X_{OUT} -> /X_{IN}
- Y1 pad 2: /X_{IN} -> GND
Routing:
- net /VDDSW: track 85.7 -> 0.00 mm, vias 2 -> 0
- net VDD: track 85.5 -> 0.00 mm, vias 3 -> 0
- net /I2C.SDA: track 54.5 -> 0.00 mm, vias 6 -> 0
- net /I2C.SCL: track 49.9 -> 0.00 mm, vias 6 -> 0
- net +5V: track 46.1 -> 1.51 mm
- net ~{RESET}: track 26.3 -> 0.00 mm
- net /CAN_{RX}: track 21.5 -> 0.00 mm
- net /CAN_{TX}: track 21.4 -> 0.00 mm
- net /SWDIO: track 17.3 -> 0.00 mm
- net /VDDSW_SIG: track 15.7 -> 0.00 mm, vias 2 -> 0
- net /5VSW_SIG: track 15.5 -> 0.00 mm, vias 2 -> 0
- net /SWCLK: track 15.4 -> 0.00 mm
- net /CAN+: track 15.0 -> 0.00 mm
- net /GPIO.1: track 13.4 -> 0.00 mm, vias 2 -> 0
- net /GPIO.0: track 12.9 -> 0.00 mm, vias 2 -> 0
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Other:
- board size 54 x 34 mm -> 50 x 34 mm

Commit message: updated pcb
Parts:
- added D2: MMBZ15VALT1G, Package_TO_SOT_SMD:SOT-23, F.Cu at (14.8, 12.4)
- added Q3: BSH203,215, Package_TO_SOT_SMD:SOT-23, F.Cu at (10.8, 12.4)
- added R10: 4k7, Resistor_SMD:R_0402_1005Metric, F.Cu at (38.6, 5.05)
- added R11: 4k7, Resistor_SMD:R_0402_1005Metric, F.Cu at (38.6, 2.80)
- added R9: 100k, Resistor_SMD:R_0402_1005Metric, F.Cu at (11.2, 14.7)
- added TP2: SDA, TestPoint:TestPoint_Pad_D1.0mm, F.Cu at (31.1, 15.4)
- added TP3: SCL, TestPoint:TestPoint_Pad_D1.0mm, F.Cu at (26.1, 12.3)
- REF** (x4): value MountingHole_3.2mm_M3 -> MountingHole_3.2mm_M3_no_Mask; footprint MountingHole:MountingHole_3.2mm_M3 -> ownLib:MountingHole_3.2mm_M3_no_Mask
- moved C13 8.76 mm to (24.6, 3.30)
- moved C12 8.76 mm to (18.8, 3.00)
- moved U3 8.76 mm to (21.7, 3.50)
- moved C10 5.73 mm to (10.9, 7.20)
- moved C11 5.73 mm to (8.90, 7.20)
- moved U4 5.73 mm to (14.3, 7.20)
- moved C14 5.73 mm to (18.3, 7.40)
- moved C15 5.73 mm to (19.3, 7.40)
- moved C16 5.73 mm to (17.3, 7.40)
- moved TP1 3.56 mm to (21.6, 11.8), turned to -90 degrees
- moved R1 3.16 mm to (9.65, 29.0), turned to 90 degrees
- moved C7 2.09 mm to (28.2, 20.7)
- moved Y1 2.09 mm to (23.8, 21.2)
- moved C5 2.09 mm to (25.2, 30.6)
- moved C4 2.09 mm to (25.8, 29.4)
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Connections:
- J2 pad 2: +36V -> Net-(J2-Pad2)
- J3 pad 2: /GPIO.0 -> /5VSW
- J3 pad 3: /GPIO.1 -> /VDDSW
- J3 pad 4: /VDDSW -> /GPIO.0
- J3 pad 5: /5VSW -> /GPIO.1
- U1 pad 1: /GPIO.0 -> /5VSW_SIG
- U1 pad 2: /GPIO.1 -> /VDDSW_SIG
- U1 pad 3: /5VSW_SIG -> /GPIO.0
- U1 pad 4: /VDDSW_SIG -> /GPIO.1
Routing:
- net /VDDSW: track 0.00 -> 110.3 mm, vias 0 -> 4
- net VDD: track 0.00 -> 100.4 mm, vias 0 -> 4
- net /I2C.SDA: track 0.00 -> 52.2 mm, vias 0 -> 6
- net +5V: track 1.51 -> 52.4 mm, vias 0 -> 2
- net /I2C.SCL: track 0.00 -> 50.2 mm, vias 0 -> 6
- net GND: track 0.00 -> 39.8 mm, vias 0 -> 104
- net /SERCOM0.3: track 0.00 -> 22.1 mm
- net /SERCOM0.2: track 0.00 -> 21.9 mm
- net /SERCOM0.1: track 0.00 -> 21.7 mm
- net /SERCOM0.0: track 0.00 -> 20.2 mm
- net /GPIO.1: track 0.00 -> 20.0 mm
- net /SWCLK: track 0.00 -> 20.0 mm
- net /SWDIO: track 0.00 -> 19.8 mm
- net /GPIO.0: track 0.00 -> 19.8 mm
- net ~{RESET}: track 0.00 -> 18.7 mm
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
Commit message: finished board
Parts:
- added G***: LOGO, ownLib:ownLogoNew, F.Cu at (12.6, 2.80)
- added REF**: OSHW-Logo2_7.3x6mm_SilkScreen, Symbol:OSHW-Logo2_7.3x6mm_SilkScreen, B.Cu at (36.0, 28.5)
- D1: value RCLAMP0502BA -> PESD2CAN; footprint Package_TO_SOT_SMD:SOT-416 -> Package_TO_SOT_SMD:SOT-23
- moved R9 6.32 mm to (17.3, 13.0), turned to -90 degrees
- moved R8 1.81 mm to (12.7, 17.0)
- moved C9 1.80 mm to (23.2, 16.9)
- moved C8 1.80 mm to (21.9, 16.9)
- moved U2 1.80 mm to (17.6, 16.9)
- moved D1 1.44 mm to (9.65, 17.0)
Connections:
- J2 pad 2: Net-(J2-Pad2) -> /CAN-
- J2 pad 3: /CAN- -> /CAN+
- J2 pad 4: /CAN+ -> Net-(J2-Pad4)
- Q3 pad 3: Net-(J2-Pad2) -> Net-(J2-Pad4)
Routing:
- net Net-(J2-Pad4): track 0.00 -> 11.7 mm
- net Net-(J2-Pad2): track 6.84 -> 0.00 mm
- net /CAN_{TX}: track 9.49 -> 11.5 mm
- net VDD: track 100.4 -> 98.9 mm
- net /CAN-: track 8.25 -> 9.58 mm
- net /CAN+: track 8.32 -> 9.61 mm
- net /CAN_{RX}: track 15.0 -> 16.2 mm
- net /5VSW: track 13.6 -> 12.6 mm
- net GND: track 39.8 -> 39.3 mm, vias 104 -> 103
Other:
- board text added: "CAN Pin: 1 GND 2 CAN Low 3 CAN High 4 Vcc"
- board text added: "github.com/useless-branch - 2021"
- board text added: "incuSens"
- board text added: "sensOut Pin: 1 GND 2 5V 3 3.3V 4 GPIO0 5 GPIO1 6 SERCOM0 7 SERCOM1 8 SERCOM2 9 SERCOM3 10 GND"

Commit message: researched parts
Parts:
- C14, C15, C16: footprint Capacitor_SMD:C_0402_1005Metric -> Capacitor_SMD:C_0603_1608Metric
- J2: footprint Connector_Molex:Molex_PicoBlade_53261-0471_1x04-1MP_P1.25mm_Horizontal -> Connector_Molex:Molex_PicoBlade_53047-0410_1x04_P1.25mm_Vertical
- moved J2 2.16 mm to (5.08, 15.1)
- moved C15 1.06 mm to (20.4, 7.38)
- moved C14 0.54 mm to (18.8, 7.39)
Routing:
- net /CAN+: track 9.61 -> 11.3 mm
- net /CAN-: track 9.58 -> 10.9 mm
- net +5V: track 52.4 -> 53.5 mm
- net Net-(J2-Pad4): track 11.7 -> 12.4 mm
- net GND: track 39.3 -> 38.7 mm, vias 103 -> 102
