File: hardware/sensor_board/Sensors.kicad_sch (KiCad schematic)
At the start: 16 parts, among them J3 Conn_01x10_MountingPin, U5 SHT30-DIS, U6 BMP384, U7 SCD4x, U8 SGP30, U9 BH1751FVI

Commit message: updated pcb
Parts:
- added R10, R11: 4k7, Resistor_SMD:R_0402_1005Metric, symbol Device:R
- added TP2: SDA, TestPoint:TestPoint_Pad_D1.0mm, symbol Connector:TestPoint
- added TP3: SCL, TestPoint:TestPoint_Pad_D1.0mm, symbol Connector:TestPoint
Connections:
- net 5V_{SW}: now also J3.2 (Pin_2); no longer J3.5 (Pin_5)
- net GPIO.0: now also J3.4 (Pin_4); no longer J3.2 (Pin_2)
- net GPIO.1: now also J3.5 (Pin_5); no longer J3.3 (Pin_3)
- net SCL: now also R10.2, TP3.1
- net SDA: now also R11.2, TP2.1
- net VDD_{SW}: now also J3.3 (Pin_3), R10.1, R11.1; no longer J3.4 (Pin_4)

Commit message: researched parts
Parts:
- C17, C18, C19, C20, C22, C23, C24, C25, C26: MOUSER_NO (none) -> 81-GCJ188R71H104KA2D
- C21: MOUSER_NO (none) -> 81-GRM188R60J106ME4D
- J3: MOUSER_NO (none) -> 538-53261-1071
- R10, R11, TP2, TP3, U7: MOUSER_NO (none) -> DO NOT ORDER
- U5: MOUSER_NO (none) -> 403-SHT30-DIS-F
- U6: MOUSER_NO (none) -> 262-BMP384
- U8: MOUSER_NO (none) -> 403-SGP30-2.5K
- U9: MOUSER_NO (none) -> 755-BH1751FVI-TR
Changed lines of the file:
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@@
 (kicad_sch (version 20210621) (generator eeschema)
   (paper "A4")
-  (junction (at 213.36 27.94) (diameter 0) (color 0 0 0 0))
   (junction (at 231.14 71.755) (diameter 0) (color 0 0 0 0))
   (junction (at 231.14 57.15) (diameter 0) (color 0 0 0 0))
   (junction (at 223.52 39.37) (diameter 0) (color 0 0 0 0))
   (junction (at 240.03 69.215) (diameter 0) (color 0 0 0 0))
+  (junction (at 213.36 27.94) (diameter 0) (color 0 0 0 0))
   (no_connect (at 58.42 76.2))
   (no_connect (at 48.26 33.02))
@@
     )
     (property "Datasheet" "" (id 3) (at 168.91 30.48 0)
+      (effects (font (size 1.27 1.27)) hide)
+    )
+    (property "MOUSER_NO" "403-SGP30-2.5K" (id 4) (at 168.91 30.48 0)
       (effects (font (size 1.27 1.27)) hide)
     )
@@
     )
     (property "Datasheet" "https://www.sensirion.com/fileadmin/user_upload/customers/sensirion/Dokumente/9.5_CO2/Sensirion_CO2_Sensors_SCD4x_Datasheet.pdf" (id 3) (at 124.46 24.13 0)
+      (effects (font (size 1.27 1.27)) hide)
+    )
+    (property "MOUSER_NO" "DO NOT ORDER" (id 4) (at 123.19 33.02 0)
       (effects (font (size 1.27 1.27)) hide)
     )
@@
       (effects (font (size 1.27 1.27)) hide)
     )
+    (property "MOUSER_NO" "403-SHT30-DIS-F" (id 4) (at 38.1 30.48 0)
+      (effects (font (size 1.27 1.27)) hide)
+    )
     (pin "1")
     (pin "2")
@@
       (effects (font (size 1.27 1.27)) hide)
     )
+    (property "MOUSER_NO" "81-GCJ188R71H104KA2D" (id 4) (at 187.96 30.48 0)
+      (effects (font (size 1.27 1.27)) hide)
+    )
     (pin "1")
     (pin "2")
@@
     )
     (property "Datasheet" "~" (id 3) (at 60.96 30.48 0)
+      (effects (font (size 1.27 1.27)) hide)
+    )
+    (property "MOUSER_NO" "81-GCJ188R71H104KA2D" (id 4) (at 60.96 30.48 0)
       (effects (font (size 1.27 1.27)) hide)
     )
@@
     )
     (property "Datasheet" "~" (id 3) (at 143.51 69.85 0)
+      (effects (font (size 1.27 1.27)) hide)
+    )
+    (property "MOUSER_NO" "538-53261-1071" (id 4) (at 143.51 69.85 0)
       (effects (font (size 1.27 1.27)) hide)
     )
@@
       (effects (font (size 1.27 1.27)) hide)
     )
+    (property "MOUSER_NO" "DO NOT ORDER" (id 4) (at 231.14 63.5 0)
+      (effects (font (size 1.27 1.27)) hide)
+    )
     (pin "1")
     (pin "2")
@@
     )
     (property "Datasheet" "~" (id 3) (at 151.13 31.75 0)
+      (effects (font (size 1.27 1.27)) hide)
+    )
+    (property "MOUSER_NO" "81-GCJ188R71H104KA2D" (id 4) (at 151.13 31.75 0)
       (effects (font (size 1.27 1.27)) hide)
     )
@@
       (effects (font (size 1.27 1.27)) hide)
     )
+    (property "MOUSER_NO" "DO NOT ORDER" (id 4) (at 231.14 73.025 0)
+      (effects (font (size 1.27 1.27)) hide)
+    )
     (pin "1")
   )
@@
       (effects (font (size 1.27 1.27)) hide)
     )
+    (property "MOUSER_NO" "DO NOT ORDER" (id 4) (at 240.03 63.5 0)
+      (effects (font (size 1.27 1.27)) hide)
+    )
     (pin "1")
     (pin "2")
@@
       (effects (font (size 1.27 1.27)) hide)
     )
+    (property "MOUSER_NO" "81-GCJ188R71H104KA2D" (id 4) (at 255.27 29.21 0)
+      (effects (font (size 1.27 1.27)) hide)
+    )
     (pin "1")
     (pin "2")
@@
     )
     (property "Datasheet" "~" (id 3) (at 36.83 71.12 0)
+      (effects (font (size 1.27 1.27)) hide)
+    )
+    (property "MOUSER_NO" "81-GCJ188R71H104KA2D" (id 4) (at 36.83 71.12 0)
       (effects (font (size 1.27 1.27)) hide)
     )
@@
     )
     (property "Datasheet" "https://co.mouser.com/datasheet/2/348/ROHMS34827_1-2561481.pdf" (id 3) (at 223.52 29.21 0)
+      (effects (font (size 1.27 1.27)) hide)
+    )
+    (property "MOUSER_NO" "755-BH1751FVI-TR" (id 4) (at 223.52 29.21 0)
       (effects (font (size 1.27 1.27)) hide)
     )
@@
       (effects (font (size 1.27 1.27)) hide)
     )
+    (property "MOUSER_NO" "81-GCJ188R71H104KA2D" (id 4) (at 22.86 71.12 0)
+      (effects (font (size 1.27 1.27)) hide)
+    )
     (pin "1")
     (pin "2")
@@
     )
     (property "Datasheet" "~" (id 3) (at 243.84 29.21 0)
+      (effects (font (size 1.27 1.27)) hide)
+    )
+    (property "MOUSER_NO" "81-GCJ188R71H104KA2D" (id 4) (at 243.84 29.21 0)
       (effects (font (size 1.27 1.27)) hide)
     )
@@
       (effects (font (size 1.27 1.27)) hide)
     )
+    (property "MOUSER_NO" "DO NOT ORDER" (id 4) (at 227.33 69.215 0)
+      (effects (font (size 1.27 1.27)) hide)
+    )
     (pin "1")
   )
@@
       (effects (font (size 1.27 1.27)) hide)
     )
+    (property "MOUSER_NO" "81-GCJ188R71H104KA2D" (id 4) (at 82.55 30.48 0)
+      (effects (font (size 1.27 1.27)) hide)
+    )
     (pin "1")
     (pin "2")
@@
     )
     (property "Datasheet" "~" (id 3) (at 92.71 30.48 0)
+      (effects (font (size 1.27 1.27)) hide)
+    )
+    (property "MOUSER_NO" "81-GRM188R60J106ME4D" (id 4) (at 92.71 30.48 0)
       (effects (font (size 1.27 1.27)) hide)
     )
@@
     )
     (property "Datasheet" "~" (id 3) (at 102.87 30.48 0)
+      (effects (font (size 1.27 1.27)) hide)
+    )
+    (property "MOUSER_NO" "81-GCJ188R71H104KA2D" (id 4) (at 102.87 30.48 0)
       (effects (font (size 1.27 1.27)) hide)
     )
@@
       (effects (font (size 1.27 1.27)) hide)
     )
+    (property "MOUSER_NO" "262-BMP384" (id 4) (at 67.31 71.12 0)
+      (effects (font (size 1.27 1.27)) hide)
+    )

Commit message: some stuff!
Parts:
- renumbered C17 to C19, C18 to C20, C19 to C21, C20 to C22, C21 to C23, C22 to C24, C23 to C25, C24 to C26, C25 to C27, C26 to C28
Changed lines of the file:
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@@
 (kicad_sch (version 20210621) (generator eeschema)
   (paper "A4")
+  (junction (at 231.14 57.15) (diameter 0) (color 0 0 0 0))
   (junction (at 240.03 69.215) (diameter 0) (color 0 0 0 0))
   (junction (at 231.14 71.755) (diameter 0) (color 0 0 0 0))
-  (junction (at 231.14 57.15) (diameter 0) (color 0 0 0 0))
   (junction (at 213.36 27.94) (diameter 0) (color 0 0 0 0))
   (junction (at 223.52 39.37) (diameter 0) (color 0 0 0 0))
@@
   (symbol (lib_id "Device:C") (at 187.96 30.48 0) (unit 1)
     (in_bom yes) (on_board yes)
-    (property "Reference" "C24" (id 0) (at 186.69 41.9099 0)
+    (property "Reference" "C26" (id 0) (at 186.69 41.9099 0)
       (effects (font (size 1.27 1.27)) (justify left))
     )
@@
   (symbol (lib_id "Device:C") (at 60.96 30.48 0) (unit 1)
     (in_bom yes) (on_board yes)
-    (property "Reference" "C19" (id 0) (at 59.69 41.9099 0)
+    (property "Reference" "C21" (id 0) (at 59.69 41.9099 0)
       (effects (font (size 1.27 1.27)) (justify left))
     )
@@
   (symbol (lib_id "Device:C") (at 151.13 31.75 0) (unit 1)
     (in_bom yes) (on_board yes)
-    (property "Reference" "C23" (id 0) (at 149.86 43.1799 0)
+    (property "Reference" "C25" (id 0) (at 149.86 43.1799 0)
       (effects (font (size 1.27 1.27)) (justify left))
     )
@@
   (symbol (lib_id "Device:C") (at 255.27 29.21 0) (unit 1)
     (in_bom yes) (on_board yes)
-    (property "Reference" "C26" (id 0) (at 254 40.6399 0)
+    (property "Reference" "C28" (id 0) (at 254 40.6399 0)
       (effects (font (size 1.27 1.27)) (justify left))
     )
@@
   (symbol (lib_id "Device:C") (at 36.83 71.12 0) (unit 1)
     (in_bom yes) (on_board yes)
-    (property "Reference" "C18" (id 0) (at 35.56 82.5499 0)
+    (property "Reference" "C20" (id 0) (at 35.56 82.5499 0)
       (effects (font (size 1.27 1.27)) (justify left))
     )
@@
   (symbol (lib_id "Device:C") (at 22.86 71.12 0) (unit 1)
     (in_bom yes) (on_board yes)
-    (property "Reference" "C17" (id 0) (at 21.59 82.5499 0)
+    (property "Reference" "C19" (id 0) (at 21.59 82.5499 0)
       (effects (font (size 1.27 1.27)) (justify left))
     )
@@
   (symbol (lib_id "Device:C") (at 243.84 29.21 0) (unit 1)
     (in_bom yes) (on_board yes)
-    (property "Reference" "C25" (id 0) (at 242.57 40.6399 0)
+    (property "Reference" "C27" (id 0) (at 242.57 40.6399 0)
       (effects (font (size 1.27 1.27)) (justify left))
     )
@@
   (symbol (lib_id "Device:C") (at 82.55 30.48 0) (unit 1)
     (in_bom yes) (on_board yes)
-    (property "Reference" "C20" (id 0) (at 81.28 41.9099 0)
+    (property "Reference" "C22" (id 0) (at 81.28 41.9099 0)
       (effects (font (size 1.27 1.27)) (justify left))
     )
@@
   (symbol (lib_id "Device:C") (at 92.71 30.48 0) (unit 1)
     (in_bom yes) (on_board yes)
-    (property "Reference" "C21" (id 0) (at 91.44 41.9099 0)
+    (property "Reference" "C23" (id 0) (at 91.44 41.9099 0)
       (effects (font (size 1.27 1.27)) (justify left))
     )
@@
   (symbol (lib_id "Device:C") (at 102.87 30.48 0) (unit 1)
     (in_bom yes) (on_board yes)
-    (property "Reference" "C22" (id 0) (at 101.6 41.9099 0)
-      (effects (font (size 1.27 1.27)) (justify left))
-    )
+    (property "Reference" "C24" (id 0) (at 101.6 41.9099 0)
+      (effects (font (size 1.27 1.27)) (justify left))
+    )
